File: potproto.sch (KiCad schematic (older format))
At the start: 14 parts, among them J1 Conn_01x02_Female, J2 Conn_01x02_Female, J3 Conn_01x02_Female, J4 Conn_01x02_Female, J5 Conn_01x06_Female, J6 Conn_01x06_Female, J7 Conn_01x06_Female, J8 Conn_01x06_Female

Commit message: rev2 BEST WITH AFTERDARK
Parts:
- removed J1, J2, J3, J4: Conn_01x02_Female, Connector_PinSocket_2.54mm:PinSocket_1x02_P2.54mm_Vertical, symbol Connector:Conn_01x02_Female
- removed J5, J6, J7, J8: Conn_01x06_Female, Connector_PinSocket_2.54mm:PinSocket_1x06_P2.54mm_Vertical, symbol Connector:Conn_01x06_Female
- added J1, J2: Conn_01x08_Male, Connector_PinHeader_2.54mm:PinHeader_1x08_P2.54mm_Vertical, symbol Connector:Conn_01x08_Male
- RV1, RV2: footprint Potentiometer_THT:Potentiometer_Alpha_RD901F-40-00D_Single_Vertical -> Potentiometer_THT:Potentiometer_Alps_RK09K_Single_Vertical
Connections:
- wire segments 56 -> 43
Changed lines of the file:
@@
 $EndDescr
-$Comp
-L power:GND #PWR02
-U 1 1 5FC6AE2E
-P 2500 4450
-F 0 "#PWR02" H 2500 4200 50  0001 C CNN
-F 1 "GND" H 2505 4277 50  0000 C CNN
-F 2 "" H 2500 4450 50  0001 C CNN
-F 3 "" H 2500 4450 50  0001 C CNN
-	1    2500 4450
-	-1   0    0    1
-$EndComp
-$Comp
-L power:+3.3V #PWR01
-U 1 1 5FC6B807
-P 2150 4450
-F 0 "#PWR01" H 2150 4300 50  0001 C CNN
-F 1 "+3.3V" H 2165 4623 50  0000 C CNN
-F 2 "" H 2150 4450 50  0001 C CNN
-F 3 "" H 2150 4450 50  0001 C CNN
-	1    2150 4450
-	1    0    0    -1
-$EndComp
-$Comp
-L Connector:Conn_01x02_Female J1
-U 1 1 5FC70DBC
-P 2350 4850
-F 0 "J1" V 2196 4898 50  0000 L CNN
-F 1 "Conn_01x02_Female" V 2287 4898 50  0000 L CNN
-F 2 "Connector_PinSocket_2.54mm:PinSocket_1x02_P2.54mm_Vertical" H 2350 4850 50  0001 C CNN
-F 3 "~" H 2350 4850 50  0001 C CNN
-	1    2350 4850
-	0    1    1    0
-$EndComp
 $Comp
 L power:GND #PWR03
@@
 Wire Wire Line
 	3950 3450 4200 3450
-Wire Wire Line
-	2500 4450 2500 4650
-Wire Wire Line
-	2500 4650 2350 4650
-Wire Wire Line
-	2150 4450 2150 4650
-Wire Wire Line
-	2150 4650 2250 4650
-$Comp
-L Connector:Conn_01x06_Female J5
-U 1 1 5FC6DFF0
-P 6150 5100
-F 0 "J5" V 5996 5348 50  0000 L CNN
-F 1 "Conn_01x06_Female" V 6087 5348 50  0000 L CNN
-F 2 "Connector_PinSocket_2.54mm:PinSocket_1x06_P2.54mm_Vertical" H 6150 5100 50  0001 C CNN
-F 3 "~" H 6150 5100 50  0001 C CNN
-	1    6150 5100
-	0    -1   1    0
-$EndComp
-$Comp
-L Connector:Conn_01x06_Female J6
-U 1 1 5FC6E9A0
-P 6150 5900
-F 0 "J6" V 5996 6148 50  0000 L CNN
-F 1 "Conn_01x06_Female" V 6087 6148 50  0000 L CNN
-F 2 "Connector_PinSocket_2.54mm:PinSocket_1x06_P2.54mm_Vertical" H 6150 5900 50  0001 C CNN
-F 3 "~" H 6150 5900 50  0001 C CNN
-	1    6150 5900
-	0    -1   1    0
-$EndComp
 $Comp
 L Device:R_POT RV1
@@
 F 0 "RV1" V 3593 3450 50  0000 C CNN
 F 1 "R_POT" V 3684 3450 50  0000 C CNN
-F 2 "Potentiometer_THT:Potentiometer_Alpha_RD901F-40-00D_Single_Vertical" H 3800 3450 50  0001 C CNN
+F 2 "Potentiometer_THT:Potentiometer_Alps_RK09K_Single_Vertical" H 3800 3450 50  0001 C CNN
 F 3 "~" H 3800 3450 50  0001 C CNN
 	1    3800 3450
@@
 F 0 "RV2" V 4743 3400 50  0000 C CNN
 F 1 "R_POT" V 4834 3400 50  0000 C CNN
-F 2 "Potentiometer_THT:Potentiometer_Alpha_RD901F-40-00D_Single_Vertical" H 4950 3400 50  0001 C CNN
+F 2 "Potentiometer_THT:Potentiometer_Alps_RK09K_Single_Vertical" H 4950 3400 50  0001 C CNN
 F 3 "~" H 4950 3400 50  0001 C CNN
 	1    4950 3400
@@
 Wire Wire Line
 	6250 4450 6250 4900
-Wire Wire Line
-	7950 3600 7950 4650
-Wire Wire Line
-	7950 4650 6350 4650
-Wire Wire Line
-	6350 4650 6350 4900
-Wire Wire Line
-	9000 3600 9000 4900
-Wire Wire Line
-	9000 4900 6450 4900
-Wire Wire Line
-	5950 4900 5950 5700
+$Comp
+L Connector:Conn_01x08_Male J1
+U 1 1 5FD97735
+P 6250 5100
+F 0 "J1" V 6177 5028 50  0000 C CNN
+F 1 "Conn_01x08_Male" V 6086 5028 50  0000 C CNN
+F 2 "Connector_PinHeader_2.54mm:PinHeader_1x08_P2.54mm_Vertical" H 6250 5100 50  0001 C CNN
+F 3 "~" H 6250 5100 50  0001 C CNN
+	1    6250 5100
+	0    -1   -1   0
+$EndComp
+Wire Wire Line
+	7950 3600 7950 4500
+Wire Wire Line
+	7950 4500 6350 4500
+Wire Wire Line
+	6350 4500 6350 4900
+Wire Wire Line
+	9000 3600 9000 4550
+Wire Wire Line
+	9000 4550 6450 4550
+Wire Wire Line
+	6450 4550 6450 4900
+Wire Wire Line
+	6550 4900 6550 4700
+Wire Wire Line
+	6550 4700 7150 4700
+Wire Wire Line
+	6650 4900 6900 4900
+Wire Wire Line
+	6900 4900 6900 5000
+$Comp
+L power:GND #PWR0101
+U 1 1 5FD9F1F7
+P 6900 5000
+F 0 "#PWR0101" H 6900 4750 50  0001 C CNN
+F 1 "GND" H 6905 4827 50  0000 C CNN
+F 2 "" H 6900 5000 50  0001 C CNN
+F 3 "" H 6900 5000 50  0001 C CNN
+	1    6900 5000
+	1    0    0    -1
+$EndComp
+$Comp
+L power:+3.3V #PWR0102
+U 1 1 5FD9F972
+P 7150 4700
+F 0 "#PWR0102" H 7150 4550 50  0001 C CNN
+F 1 "+3.3V" V 7165 4828 50  0000 L CNN
+F 2 "" H 7150 4700 50  0001 C CNN
+F 3 "" H 7150 4700 50  0001 C CNN
+	1    7150 4700
+	0    1    1    0
+$EndComp
+$Comp
+L Connector:Conn_01x08_Male J2
+U 1 1 5FDA044D
+P 6250 5750
+F 0 "J2" V 6177 5678 50  0000 C CNN
+F 1 "Conn_01x08_Male" V 6086 5678 50  0000 C CNN
+F 2 "Connector_PinHeader_2.54mm:PinHeader_1x08_P2.54mm_Vertical" H 6250 5750 50  0001 C CNN
+F 3 "~" H 6250 5750 50  0001 C CNN
+	1    6250 5750
+	0    -1   -1   0
+$EndComp
+$Comp
+L power:+3.3V #PWR0103
+U 1 1 5FDA5088
+P 7200 5350
+F 0 "#PWR0103" H 7200 5200 50  0001 C CNN
+F 1 "+3.3V" V 7215 5478 50  0000 L CNN
+F 2 "" H 7200 5350 50  0001 C CNN
+F 3 "" H 7200 5350 50  0001 C CNN
+	1    7200 5350
+	0    1    1    0
+$EndComp
+$Comp
+L power:GND #PWR0104
+U 1 1 5FDA5973
+P 6850 5700
+F 0 "#PWR0104" H 6850 5450 50  0001 C CNN
+F 1 "GND" H 6855 5527 50  0000 C CNN
+F 2 "" H 6850 5700 50  0001 C CNN
+F 3 "" H 6850 5700 50  0001 C CNN
+	1    6850 5700
+	1    0    0    -1
+$EndComp
+Connection ~ 6450 4900
+Wire Wire Line
+	6350 4900 6350 5550
+Wire Wire Line
+	6450 4900 6450 5550
+Connection ~ 6350 4900
+Wire Wire Line
+	6250 4900 6250 5550
+Connection ~ 6250 4900
+Wire Wire Line
+	6150 4900 6150 5550
+Connection ~ 6150 4900
+Wire Wire Line
+	6050 4900 6050 5550
+Connection ~ 6050 4900
+Wire Wire Line
+	5950 4900 5950 5550
 Connection ~ 5950 4900
 Wire Wire Line
-	6050 4900 6050 5700
-Connection ~ 6050 4900
-Wire Wire Line
-	6150 4900 6150 5700
-Connection ~ 6150 4900
-Wire Wire Line
-	6250 4900 6250 5700
-Connection ~ 6250 4900
-Wire Wire Line
-	6350 4900 6350 5700
-Connection ~ 6350 4900
-Wire Wire Line
-	6450 4900 6450 5700
-Connection ~ 6450 4900
-$Comp
-L Connector:Conn_01x02_Female J2
-U 1 1 5FC961CB
-P 2350 5350
-F 0 "J2" V 2196 5398 50  0000 L CNN
-F 1 "Conn_01x02_Female" V 2287 5398 50  0000 L CNN
-F 2 "Connector_PinSocket_2.54mm:PinSocket_1x02_P2.54mm_Vertical" H 2350 5350 50  0001 C CNN
-F 3 "~" H 2350 5350 50  0001 C CNN
-	1    2350 5350
-	0    1    1    0
-$EndComp
-Wire Wire Line
-	2250 4650 2250 5150
-Connection ~ 2250 4650
-Wire Wire Line
-	2350 4650 2350 5150
-Connection ~ 2350 4650
-$Comp
-L Connector:Conn_01x02_Female J3
-U 1 1 5FCA216B
-P 2350 5800
-F 0 "J3" V 2196 5848 50  0000 L CNN
-F 1 "Conn_01x02_Female" V 2287 5848 50  0000 L CNN
-F 2 "Connector_PinSocket_2.54mm:PinSocket_1x02_P2.54mm_Vertical" H 2350 5800 50  0001 C CNN
-F 3 "~" H 2350 5800 50  0001 C CNN
-	1    2350 5800
-	0    1    1    0
-$EndComp
-$Comp
-L Connector:Conn_01x02_Female J4
-U 1 1 5FCA269C
-P 2350 6250
-F 0 "J4" V 2196 6298 50  0000 L CNN
-F 1 "Conn_01x02_Female" V 2287 6298 50  0000 L CNN
-F 2 "Connector_PinSocket_2.54mm:PinSocket_1x02_P2.54mm_Vertical" H 2350 6250 50  0001 C CNN
-F 3 "~" H 2350 6250 50  0001 C CNN
-	1    2350 6250
-	0    1    1    0
-$EndComp
-Wire Wire Line
-	2250 5150 2250 5600
-Connection ~ 2250 5150
-Wire Wire Line
-	2250 5600 2250 6050
-Connection ~ 2250 5600
-Wire Wire Line
-	2350 5150 2350 5600
-Connection ~ 2350 5150
-Wire Wire Line
-	2350 5600 2350 6050
-Connection ~ 2350 5600
-$Comp
-L Connector:Conn_01x06_Female J7
-U 1 1 5FCAA771
-P 6150 6250
-F 0 "J7" V 5996 6498 50  0000 L CNN
-F 1 "Conn_01x06_Female" V 6087 6498 50  0000 L CNN
-F 2 "Connector_PinSocket_2.54mm:PinSocket_1x06_P2.54mm_Vertical" H 6150 6250 50  0001 C CNN
-F 3 "~" H 6150 6250 50  0001 C CNN
-	1    6150 6250
-	0    -1   1    0
-$EndComp
-$Comp
-L Connector:Conn_01x06_Female J8
-U 1 1 5FCAB26C
-P 6150 6600
-F 0 "J8" V 5996 6848 50  0000 L CNN
-F 1 "Conn_01x06_Female" V 6087 6848 50  0000 L CNN
-F 2 "Connector_PinSocket_2.54mm:PinSocket_1x06_P2.54mm_Vertical" H 6150 6600 50  0001 C CNN
-F 3 "~" H 6150 6600 50  0001 C CNN
-	1    6150 6600
-	0    -1   1    0
-$EndComp
-Wire Wire Line
-	5950 5700 5950 6050
-Connection ~ 5950 5700
-Wire Wire Line
-	5950 6050 5950 6400
-Connection ~ 5950 6050
-Wire Wire Line
-	6050 5700 6050 6050
-Connection ~ 6050 5700
-Wire Wire Line
-	6050 6400 6050 6050
-Connection ~ 6050 6050
-Wire Wire Line
-	6150 5700 6150 6050
-Connection ~ 6150 5700
-Wire Wire Line
-	6150 6050 6150 6400
-Connection ~ 6150 6050
-Wire Wire Line
-	6250 5700 6250 6050
-Connection ~ 6250 5700
-Wire Wire Line
-	6250 6050 6250 6400
-Connection ~ 6250 6050
-Wire Wire Line
-	6350 5700 6350 6050
-Connection ~ 6350 5700
-Wire Wire Line
-	6350 6050 6350 6400
-Connection ~ 6350 6050
-Wire Wire Line
-	6450 5700 6450 6050
-Connection ~ 6450 5700
-Wire Wire Line
-	6450 6050 6450 6400
-Connection ~ 6450 6050
+	6550 5550 6550 5350
+Wire Wire Line
+	6550 5350 7200 5350
+Wire Wire Line
+	6650 5550 6850 5550
+Wire Wire Line
+	6850 5550 6850 5700
 $EndSCHEMATC
